File: Hardware/KiCad_Stator/KiCad_Stator.kicad_pcb (KiCad board)
At the start: 2 copper layers, 40 x 40 mm, 0 parts

Commit message: feat: 9 Slot (#3)
Other:
- board size 40 x 40 mm -> 29.5 x 29.5 mm
