File: Hardware/KiCad_FOC-ESC/KiCad_FOC-ESC.kicad_pcb (KiCad board)
At the start: 2 copper layers, 41 x 41 mm, 37 parts, among them IC1 DRV8300DPWR, IC2 TSC1801BILT, IC3 TSC1801BILT, IC4 TSC1801BILT, IC5 AZ431LBNTR-G1, IC6 MA702GQ-P, Q1 NTTFS5D6N08XLTAG, Q2 10nF, Q2 NTTFS5D6N08XLTAG, Q3 NTTFS5D6N08XLTAG, Q4 100nF, Q4 NTTFS5D6N08XLTAG, Q5 NTTFS5D6N08XLTAG, Q6 1uF, U1 REF3030AIDBZR, U1 STM32G473RCTx, U3 MT6701CT, Y1 ASDDV-16.000MHZ-LR-T

Commit message: updated:schematics (#9)
Parts:
- removed the C1 at (156.4, 82.5) (x2)
- removed the C3 at (153.0, 84.2) (x2)
- removed C701: 10nF, Capacitor_SMD:C_0402_1005Metric
- removed the C8 at (156.4, 87.6) (x2)
- removed the C9 at (153.0, 92.1) (x2)
- removed the IC3 at (144.5, 96.2)
- removed the IC3 at (128.9, 99.7)
- removed the IC4 at (128.9, 104.3) (x2)
- removed IC5: AZ431LBNTR-G1, SamacSys_Parts:SOT96P240X105-3N
- removed the Q2 at (144.2, 103.4)
- removed the Q2 at (137.3, 106.7)
- removed the Q4 at (137.9, 109.7)
- removed the Q4 at (144.5, 109.7)
- removed the U1 at (144.0, 84.2) (x2)
- removed the Y1 at (158.4, 93.4)
- removed the Y1 at (158.4, 92.4)
- added C1: 4.7uF, Capacitor_SMD:C_0603_1608Metric, F.Cu at (94.8, 85.8)
- added C10: 100nF, Capacitor_SMD:C_0402_1005Metric, F.Cu at (197.2, 95.2)
- added C11: 100nF, Capacitor_SMD:C_0402_1005Metric, F.Cu at (205.1, 95.2)
- added C12: 100nF, Capacitor_SMD:C_0402_1005Metric, F.Cu at (213.0, 95.2)
- added C3: 100nF, Capacitor_SMD:C_0402_1005Metric, F.Cu at (91.4, 87.5)
- added C8: 1uF, Capacitor_SMD:C_0603_1608Metric, F.Cu at (94.8, 90.8)
- added C9: 100nF, Capacitor_SMD:C_0402_1005Metric, F.Cu at (91.4, 95.3)
- added IC3: TSC1801BILT, SamacSys_Parts:SOT95P280X145-6N, F.Cu at (205.6, 97.8)
- added IC4: TSC1801BILT, SamacSys_Parts:SOT95P280X145-6N, F.Cu at (213.5, 97.8)
- added J1: Conn_01x01_Socket, Connector_PinHeader_2.54mm:PinHeader_1x01_P2.54mm_Vertical, F.Cu at (197.2, 109.5)
- added J2: Conn_01x01_Socket, Connector_PinHeader_2.54mm:PinHeader_1x01_P2.54mm_Vertical, F.Cu at (205.1, 109.5)
- added J3: Conn_01x01_Socket, Connector_PinHeader_2.54mm:PinHeader_1x01_P2.54mm_Vertical, F.Cu at (213.0, 109.5)
- added PS1: REF3030AIDBZR, SamacSys_Parts:SOT96P240X105-3N, F.Cu at (105.3, 112.4)
- added Q2: NTTFS5D6N08XLTAG, SamacSys_Parts:NVTFS007N08HLTAG, F.Cu at (195.3, 105.4)
- added Q4: NTTFS5D6N08XLTAG, SamacSys_Parts:NVTFS007N08HLTAG, F.Cu at (203.2, 105.4)
- added R4: PMR25HZPFV1L00, SamacSys_Parts:RESC3225X67N, F.Cu at (197.2, 101.6)
- added R5: PMR25HZPFV1L00, SamacSys_Parts:RESC3225X67N, F.Cu at (205.1, 101.6)
- added R6: PMR25HZPFV1L00, SamacSys_Parts:RESC3225X67N, F.Cu at (213.0, 101.6)
- added U1: STM32G473RCTx, Package_QFP:LQFP-64_10x10mm_P0.5mm, F.Cu at (205.6, 72.1)
- added Y1: ASDDV-16.000MHZ-LR-T, SamacSys_Parts:AbraconASDDV, F.Cu at (106.2, 102.0)
- Q6: value 1uF -> NTTFS5D6N08XLTAG; footprint Capacitor_SMD:C_0603_1608Metric -> SamacSys_Parts:NVTFS007N08HLTAG
- moved Q5 72.9 mm to (214.9, 105.5), turned to 0 degrees
- moved IC1 72.7 mm to (205.6, 85.0), turned to -90 degrees
- moved IC2 68.8 mm to (197.7, 97.8), turned to -90 degrees
- moved C2 61.7 mm to (91.4, 85.5)
- moved C4 61.7 mm to (91.4, 89.4)
- moved C5 61.7 mm to (91.4, 91.4)
- moved C6 61.7 mm to (94.8, 88.3)
- moved C7 61.7 mm to (91.4, 93.4)
- moved Q1 61.5 mm to (199.1, 105.5)
- moved Q6 60.2 mm to (211.1, 105.4), turned to 180 degrees
- moved U3 59.0 mm to (87.2, 110.6), turned to 180 degrees
- moved Q3 56.3 mm to (207.0, 105.5)
- moved C103 53.5 mm to (104.4, 107.2)
- moved IC6 53.5 mm to (93.8, 113.2)
- moved LED1 24.8 mm to (110.2, 105.2)
Connections:
- IC1 pad 1: unconnected-(IC1-INHA-Pad1) -> INHA
- IC1 pad 10: unconnected-(IC1-GLB-Pad10) -> GLB
- IC1 pad 11: unconnected-(IC1-GLA-Pad11) -> GLA
- IC1 pad 12: unconnected-(IC1-SHC-Pad12) -> SHC
- IC1 pad 13: unconnected-(IC1-GHC-Pad13) -> GHC
- IC1 pad 14: unconnected-(IC1-BSTC-Pad14) -> BSTC
- IC1 pad 15: unconnected-(IC1-SHB-Pad15) -> SHB
- IC1 pad 16: unconnected-(IC1-GHB-Pad16) -> GHB
- IC1 pad 17: unconnected-(IC1-BSTB-Pad17) -> BSTB
- IC1 pad 18: unconnected-(IC1-SHA-Pad18) -> SHA
- IC1 pad 19: unconnected-(IC1-GHA-Pad19) -> GHA
- IC1 pad 2: unconnected-(IC1-INHB-Pad2) -> INHB
- IC1 pad 20: unconnected-(IC1-BSTA-Pad20) -> BSTA
- IC1 pad 3: unconnected-(IC1-INHC-Pad3) -> INHC
- IC1 pad 4: unconnected-(IC1-INLA-Pad4) -> INLA
- IC1 pad 5: unconnected-(IC1-INLB-Pad5) -> INLB
- IC1 pad 6: unconnected-(IC1-INLC-Pad6) -> INLC
- IC1 pad 9: unconnected-(IC1-GLC-Pad9) -> GLC
- IC2 pad 1: unconnected-(IC2-VREF-Pad1) -> Vref
- IC2 pad 2: unconnected-(IC2-VCC--Pad2) -> GND
- IC2 pad 3: unconnected-(IC2-VCC+-Pad3) -> +3V3
- IC2 pad 4: unconnected-(IC2-IN+-Pad4) -> /FETs/HalfBridgeA/GND1
- IC2 pad 5: unconnected-(IC2-IN--Pad5) -> GND
- IC2 pad 6: unconnected-(IC2-OUT-Pad6) -> /FETs/HalfBridgeA/OUT
- IC6 pad 1: GND -> unconnected-(IC6-SSD-Pad1)
- IC6 pad 16: GND -> unconnected-(IC6-MGH-Pad16)
- IC6 pad 17: +3V3 -> unconnected-(IC6-GND_2-Pad17)
- LED1 pad 1: /Debbug/DO -> unconnected-(LED1-DO-Pad1)
- LED1 pad 2: GND -> unconnected-(LED1-GND-Pad2)
- LED1 pad 3: +3V3 -> unconnected-(LED1-DI-Pad3)
- LED1 pad 4: +5V -> unconnected-(LED1-VDD-Pad4)
- Q1 pad 1: unconnected-(Q6-S_1-Pad1) -> /FETs/HalfBridgeA/MP
- Q1 pad 10: unconnected-(Q6-D_6-Pad10) -> VCC
- Q1 pad 11: unconnected-(Q6-D_7-Pad11) -> VCC
- Q1 pad 12: unconnected-(Q6-S_4-Pad12) -> /FETs/HalfBridgeA/MP
- Q1 pad 2: unconnected-(Q6-S_2-Pad2) -> /FETs/HalfBridgeA/MP
- Q1 pad 3: unconnected-(Q6-S_3-Pad3) -> /FETs/HalfBridgeA/MP
- Q1 pad 4: unconnected-(Q6-G-Pad4) -> GHA
- Q1 pad 5: unconnected-(Q6-D_1-Pad5) -> VCC
- Q1 pad 6: unconnected-(Q6-D_2-Pad6) -> VCC
- Q1 pad 7: unconnected-(Q6-D_3-Pad7) -> VCC
- Q1 pad 8: unconnected-(Q6-D_4-Pad8) -> VCC
- Q1 pad 9: unconnected-(Q6-D_5-Pad9) -> VCC
- Q3 pad 1: unconnected-(Q3-S_1-Pad1) -> /FETs/HalfBridgeB/MP
- Q3 pad 10: unconnected-(Q3-D_6-Pad10) -> VCC
- Q3 pad 11: unconnected-(Q3-D_7-Pad11) -> VCC
- Q3 pad 12: unconnected-(Q3-S_4-Pad12) -> /FETs/HalfBridgeB/MP
- Q3 pad 2: unconnected-(Q3-S_2-Pad2) -> /FETs/HalfBridgeB/MP
- Q3 pad 3: unconnected-(Q3-S_3-Pad3) -> /FETs/HalfBridgeB/MP
- Q3 pad 4: unconnected-(Q3-G-Pad4) -> GHB
- Q3 pad 5: unconnected-(Q3-D_1-Pad5) -> VCC
- Q3 pad 6: unconnected-(Q3-D_2-Pad6) -> VCC
- Q3 pad 7: unconnected-(Q3-D_3-Pad7) -> VCC
- Q3 pad 8: unconnected-(Q3-D_4-Pad8) -> VCC
- Q3 pad 9: unconnected-(Q3-D_5-Pad9) -> VCC
- Q5 pad 1: unconnected-(Q5-S_1-Pad1) -> /FETs/HalfBridgeC/MP
- Q5 pad 10: unconnected-(Q5-D_6-Pad10) -> VCC
- Q5 pad 11: unconnected-(Q5-D_7-Pad11) -> VCC
- Q5 pad 12: unconnected-(Q5-S_4-Pad12) -> /FETs/HalfBridgeC/MP
- Q5 pad 2: unconnected-(Q5-S_2-Pad2) -> /FETs/HalfBridgeC/MP
- Q5 pad 3: unconnected-(Q5-S_3-Pad3) -> /FETs/HalfBridgeC/MP
- Q5 pad 4: unconnected-(Q5-G-Pad4) -> GHC
- Q5 pad 5: unconnected-(Q5-D_1-Pad5) -> VCC
- Q5 pad 6: unconnected-(Q5-D_2-Pad6) -> VCC
- Q5 pad 7: unconnected-(Q5-D_3-Pad7) -> VCC
- Q5 pad 8: unconnected-(Q5-D_4-Pad8) -> VCC
- Q5 pad 9: unconnected-(Q5-D_5-Pad9) -> VCC
- Q6 pad 1: +3V3 -> /FETs/HalfBridgeC/GND1
- Q6 pad 2: GND -> /FETs/HalfBridgeC/GND1
Routing:
- net GND: track 0.00 -> 20.2 mm
- net +3V3: track 0.00 -> 3.94 mm
- net /FETs/HalfBridgeC/GND1: track 0.00 -> 2.85 mm
- net /FETs/HalfBridgeB/GND1: track 0.00 -> 2.85 mm
- net /FETs/HalfBridgeA/GND1: track 0.00 -> 2.85 mm
- net GHC: track 0.00 -> 0.99 mm, vias 0 -> 1
- net GHB: track 0.00 -> 0.99 mm, vias 0 -> 1
- net GHA: track 0.00 -> 0.99 mm, vias 0 -> 1
- added copper zone on F.Cu, net /FETs/HalfBridgeA/GND1
- added copper zone on F.Cu, net /FETs/HalfBridgeA/MP
- added copper zone on F.Cu, net /FETs/HalfBridgeB/GND1
- added copper zone on F.Cu, net /FETs/HalfBridgeB/MP
- added copper zone on F.Cu, net /FETs/HalfBridgeC/GND1
- added copper zone on F.Cu, net /FETs/HalfBridgeC/MP
- added copper zone on F.Cu, net VCC
Other:
- copper layers 2 -> 4
